File: ECAD/PumpBoard-2026/PumpBoard-2026.kicad_pcb (KiCad board)
At the start: 2 copper layers, 30 x 28 mm, 18 parts, among them J1 Conn_01x04, J3 CON_EV, J4 CON_PUMP, Q1 AO3400A, Q2 AO3400A

Commit message: routage carte pompe
Parts:
- added G***: LOGO, LOGO, F.Cu at (138.9, 94.5)
- added kibuzzard-69769280: G***, kibuzzard-69769280, F.Cu at (126.8, 99.7)
- added kibuzzard-6976928C: G***, kibuzzard-6976928C, F.Cu at (126.7, 102.2)
- added kibuzzard-69769299: G***, kibuzzard-69769299, F.Cu at (126.6, 97.2)
- added kibuzzard-697692E7: G***, kibuzzard-697692E7, F.Cu at (137.0, 88.4)
- added kibuzzard-6976930F: G***, kibuzzard-6976930F, F.Cu at (123.4, 89.0)
- added kibuzzard-697693AB: G***, kibuzzard-697693AB, F.Cu at (136.5, 111.5)
- added kibuzzard-697693BC: G***, kibuzzard-697693BC, F.Cu at (127.0, 111.2)
- added kibuzzard-6976945E: G***, kibuzzard-6976945E, F.Cu at (124.4, 109.2)
- added kibuzzard-6976947C: G***, kibuzzard-6976947C, F.Cu at (140.9, 106.3)
- added kibuzzard-69769485: G***, kibuzzard-69769485, F.Cu at (132.6, 92.2)
- moved D4 6.31 mm to (129.0, 91.5), turned to -90 degrees
- moved Q1 1.85 mm to (132.6, 94.8)
- moved D5 1.58 mm to (144.5, 94.0), turned to -90 degrees
- moved R5 1.56 mm to (130.9, 100.5), turned to 180 degrees
- moved R7 1.56 mm to (130.9, 98.0)
- moved Q2 0.47 mm to (144.7, 107.1)
- moved R8 0.47 mm to (144.9, 103.3)
- moved R6 0.47 mm to (144.9, 100.6)
Routing:
- net +5V: track 0.00 -> 57.0 mm, vias 0 -> 1
- net S_PUMP: track 0.00 -> 25.3 mm, vias 0 -> 2
- net Net-(D5-A): track 0.00 -> 22.9 mm
- net S_EV: track 0.00 -> 10.5 mm
- net Net-(D4-A): track 0.00 -> 8.19 mm
- net Net-(Q1-G): track 0.00 -> 7.55 mm
- net Net-(Q2-G): track 0.00 -> 5.93 mm
- net Net-(D1-A): track 0.00 -> 2.04 mm
- net Net-(D2-A): track 0.00 -> 2.04 mm
- net Net-(D3-A): track 0.00 -> 2.04 mm
- net GND: vias 0 -> 4
- added copper zone on B.Cu, net GND
- added copper zone on F.Cu, net GND
Other:
- board text added: "Barbatronic"
- board text added: "Pump Board 2026"
